File: Window Detector/Window Detector.sch (KiCad schematic (older format))
At the start: 17 parts, among them J1 CONN_01X02, J2 CONN_01X03, J3 CONN_01X03, U1 LM741, U2 LM741

Commit message: Made some changes in circuit
Yet to update the changes in the pcb design
Parts:
- added R10: 6.2K, symbol R
- R9: value 6.2K -> 10K
Connections:
- net at D1.2 (A), R8.2, R9.2: now also R10.1; no longer D2.1 (K), U1.6
- new net: D2.1 (K), R10.2, U1.6
Changed lines of the file:
@@
 $EndComp
 $Comp
-L GND #PWR01
+L GND #PWR14
 U 1 1 59C81852
 P 4000 5450
-F 0 "#PWR01" H 4000 5200 50  0001 C CNN
+F 0 "#PWR14" H 4000 5200 50  0001 C CNN
 F 1 "GND" H 4000 5300 50  0000 C CNN
 F 2 "" H 4000 5450 50  0001 C CNN
@@
 $EndComp
 $Comp
-L GND #PWR02
+L GND #PWR21
 U 1 1 59C81C40
 P 6800 5500
-F 0 "#PWR02" H 6800 5250 50  0001 C CNN
+F 0 "#PWR21" H 6800 5250 50  0001 C CNN
 F 1 "GND" H 6800 5350 50  0000 C CNN
 F 2 "" H 6800 5500 50  0001 C CNN
@@
 Wire Wire Line
 	6000 4850 6000 3750
-Wire Wire Line
-	6000 2200 6000 3450
-$Comp
-L GND #PWR03
+$Comp
+L GND #PWR22
 U 1 1 59C82367
 P 6850 1500
-F 0 "#PWR03" H 6850 1250 50  0001 C CNN
+F 0 "#PWR22" H 6850 1250 50  0001 C CNN
 F 1 "GND" H 6850 1350 50  0000 C CNN
 F 2 "" H 6850 1500 50  0001 C CNN
@@
 $EndComp
 $Comp
-L PWR_FLAG #FLG04
+L PWR_FLAG #FLG2
 U 1 1 59C88EE7
 P 1850 2100
-F 0 "#FLG04" H 1850 2175 50  0001 C CNN
+F 0 "#FLG2" H 1850 2175 50  0001 C CNN
 F 1 "PWR_FLAG" H 1850 2250 50  0000 C CNN
 F 2 "" H 1850 2100 50  0001 C CNN
@@
 $EndComp
 $Comp
-L PWR_FLAG #FLG05
+L PWR_FLAG #FLG4
 U 1 1 59C88F1C
 P 2350 2100
-F 0 "#FLG05" H 2350 2175 50  0001 C CNN
+F 0 "#FLG4" H 2350 2175 50  0001 C CNN
 F 1 "PWR_FLAG" H 2350 2250 50  0000 C CNN
 F 2 "" H 2350 2100 50  0001 C CNN
@@
 Vin
 $Comp
-L +15V #PWR06
+L +15V #PWR16
 U 1 1 59C93462
 P 5250 2450
-F 0 "#PWR06" H 5250 2300 50  0001 C CNN
+F 0 "#PWR16" H 5250 2300 50  0001 C CNN
 F 1 "+15V" H 5250 2590 50  0000 C CNN
 F 2 "" H 5250 2450 50  0001 C CNN
@@
 $EndComp
 $Comp
-L +15V #PWR07
+L +15V #PWR18
 U 1 1 59C9352F
 P 5300 4100
-F 0 "#PWR07" H 5300 3950 50  0001 C CNN
+F 0 "#PWR18" H 5300 3950 50  0001 C CNN
 F 1 "+15V" H 5300 4240 50  0000 C CNN
 F 2 "" H 5300 4100 50  0001 C CNN
@@
 $EndComp
 $Comp
-L +15V #PWR08
+L +15V #PWR1
 U 1 1 59C93C04
 P 1850 2100
-F 0 "#PWR08" H 1850 1950 50  0001 C CNN
+F 0 "#PWR1" H 1850 1950 50  0001 C CNN
 F 1 "+15V" H 1850 2240 50  0000 C CNN
 F 2 "" H 1850 2100 50  0001 C CNN
@@
 $EndComp
 $Comp
-L PWR_FLAG #FLG09
+L PWR_FLAG #FLG1
 U 1 1 59C93C33
 P 1850 1450
-F 0 "#FLG09" H 1850 1525 50  0001 C CNN
+F 0 "#FLG1" H 1850 1525 50  0001 C CNN
 F 1 "PWR_FLAG" H 1850 1600 50  0000 C CNN
 F 2 "" H 1850 1450 50  0001 C CNN
@@
 Vin
 $Comp
-L PWR_FLAG #FLG010
+L PWR_FLAG #FLG3
 U 1 1 59C93C88
 P 2350 1450
-F 0 "#FLG010" H 2350 1525 50  0001 C CNN
+F 0 "#FLG3" H 2350 1525 50  0001 C CNN
 F 1 "PWR_FLAG" H 2350 1600 50  0000 C CNN
 F 2 "" H 2350 1450 50  0001 C CNN
@@
 $EndComp
 $Comp
-L +9V #PWR011
+L +9V #PWR13
 U 1 1 59C93DDA
 P 4000 1700
-F 0 "#PWR011" H 4000 1550 50  0001 C CNN
+F 0 "#PWR13" H 4000 1550 50  0001 C CNN
 F 1 "+9V" H 4000 1840 50  0000 C CNN
 F 2 "" H 4000 1700 50  0001 C CNN
@@
 $EndComp
 $Comp
-L +9V #PWR012
+L +9V #PWR2
 U 1 1 59C93E10
 P 2350 1450
-F 0 "#PWR012" H 2350 1300 50  0001 C CNN
+F 0 "#PWR2" H 2350 1300 50  0001 C CNN
 F 1 "+9V" H 2350 1590 50  0000 C CNN
 F 2 "" H 2350 1450 50  0001 C CNN
@@
 $EndComp
 $Comp
-L +15V #PWR013
+L +15V #PWR7
 U 1 1 59C94667
 P 2850 4150
-F 0 "#PWR013" H 2850 4000 50  0001 C CNN
+F 0 "#PWR7" H 2850 4000 50  0001 C CNN
 F 1 "+15V" H 2850 4290 50  0000 C CNN
 F 2 "" H 2850 4150 50  0001 C CNN
@@
 	2750 3900 3000 3900
 $Comp
-L GND #PWR014
+L GND #PWR4
 U 1 1 59C94947
 P 2750 3600
-F 0 "#PWR014" H 2750 3350 50  0001 C CNN
+F 0 "#PWR4" H 2750 3350 50  0001 C CNN
 F 1 "GND" H 2750 3450 50  0000 C CNN
 F 2 "" H 2750 3600 50  0001 C CNN
@@
 $EndComp
 $Comp
-L PWR_FLAG #FLG015
+L PWR_FLAG #FLG5
 U 1 1 59C94D82
 P 2950 1450
-F 0 "#FLG015" H 2950 1525 50  0001 C CNN
+F 0 "#FLG5" H 2950 1525 50  0001 C CNN
 F 1 "PWR_FLAG" H 2950 1600 50  0000 C CNN
 F 2 "" H 2950 1450 50  0001 C CNN
@@
 $EndComp
 $Comp
-L -9VA #PWR016
+L -9VA #PWR8
 U 1 1 59C94DA9
 P 2950 1450
-F 0 "#PWR016" H 2950 1325 50  0001 C CNN
+F 0 "#PWR8" H 2950 1325 50  0001 C CNN
 F 1 "-9VA" H 2950 1600 50  0000 C CNN
 F 2 "" H 2950 1450 50  0001 C CNN
@@
 $EndComp
 $Comp
-L -9VA #PWR017
+L -9VA #PWR15
 U 1 1 59C94DE5
 P 5000 5500
-F 0 "#PWR017" H 5000 5375 50  0001 C CNN
+F 0 "#PWR15" H 5000 5375 50  0001 C CNN
 F 1 "-9VA" H 5000 5650 50  0000 C CNN
 F 2 "" H 5000 5500 50  0001 C CNN
@@
 $EndComp
 $Comp
-L GND #PWR018
+L GND #PWR9
 U 1 1 59C956A3
 P 2950 2650
-F 0 "#PWR018" H 2950 2400 50  0001 C CNN
+F 0 "#PWR9" H 2950 2400 50  0001 C CNN
 F 1 "GND" H 2950 2500 50  0000 C CNN
 F 2 "" H 2950 2650 50  0001 C CNN
@@
 	3200 4900 2750 4900
 $Comp
-L +9V #PWR019
+L +9V #PWR6
 U 1 1 59C95847
 P 2750 5400
-F 0 "#PWR019" H 2750 5250 50  0001 C CNN
+F 0 "#PWR6" H 2750 5250 50  0001 C CNN
 F 1 "+9V" H 2750 5540 50  0000 C CNN
 F 2 "" H 2750 5400 50  0001 C CNN
@@
 $EndComp
 $Comp
-L -9VA #PWR020
+L -9VA #PWR12
 U 1 1 59C9587F
 P 3200 5000
-F 0 "#PWR020" H 3200 4875 50  0001 C CNN
+F 0 "#PWR12" H 3200 4875 50  0001 C CNN
 F 1 "-9VA" H 3200 5150 50  0000 C CNN
 F 2 "" H 3200 5000 50  0001 C CNN
@@
 	2950 2950 2950 2650
 $Comp
-L GND #PWR021
+L GND #PWR5
 U 1 1 59C95A91
 P 2750 4600
-F 0 "#PWR021" H 2750 4350 50  0001 C CNN
+F 0 "#PWR5" H 2750 4350 50  0001 C CNN
 F 1 "GND" H 2750 4450 50  0000 C CNN
 F 2 "" H 2750 4600 50  0001 C CNN
@@
 	3200 5000 3200 4900
 $Comp
-L PWR_FLAG #FLG022
+L PWR_FLAG #FLG6
 U 1 1 59C95B37
 P 3000 2100
-F 0 "#FLG022" H 3000 2175 50  0001 C CNN
+F 0 "#FLG6" H 3000 2175 50  0001 C CNN
 F 1 "PWR_FLAG" H 3000 2250 50  0000 C CNN
 F 2 "" H 3000 2100 50  0001 C CNN
@@
 $EndComp
 $Comp
-L GND #PWR023
+L GND #PWR10
 U 1 1 59C95B6F
 P 3000 2100
-F 0 "#PWR023" H 3000 1850 50  0001 C CNN
+F 0 "#PWR10" H 3000 1850 50  0001 C CNN
 F 1 "GND" H 3000 1950 50  0000 C CNN
 F 2 "" H 3000 2100 50  0001 C CNN
@@
 P 6400 2400
 F 0 "R9" V 6480 2400 50  0000 C CNN
-F 1 "6.2K" V 6400 2400 50  0000 C CNN
+F 1 "10K" V 6400 2400 50  0000 C CNN
 F 2 "Resistors_THT:R_Axial_DIN0207_L6.3mm_D2.5mm_P15.24mm_Horizontal" V 6330 2400 50  0001 C CNN
 F 3 "" H 6400 2400 50  0001 C CNN
@@
 	6750 2400 6750 2700
 $Comp
-L GND #PWR024
+L GND #PWR20
 U 1 1 59CD77EA
 P 6750 2700
-F 0 "#PWR024" H 6750 2450 50  0001 C CNN
+F 0 "#PWR20" H 6750 2450 50  0001 C CNN
 F 1 "GND" H 6750 2550 50  0000 C CNN
 F 2 "" H 6750 2700 50  0001 C CNN
@@
 	1    0    0    -1
 $EndComp
+$Comp
+L R R10
+U 1 1 59D3CC94
+P 6000 2550
+F 0 "R10" V 6080 2550 50  0000 C CNN
+F 1 "6.2K" V 6000 2550 50  0000 C CNN
+F 2 "" V 5930 2550 50  0001 C CNN
+F 3 "" H 6000 2550 50  0001 C CNN
+	1    6000 2550
+	1    0    0    -1
+$EndComp
+Wire Wire Line
+	6000 2200 6000 2400
+Wire Wire Line
+	6000 2700 6000 3450
 $EndSCHEMATC
