File: Class_C_Commutation/Class_C_Commuttation_Schematic.sch (KiCad schematic (older format))
At the start: 16 parts, among them J1 CONN_01X01, J2 CONN_01X01, J3 CONN_01X01, J4 CONN_01X01

Commit message: Class C commutation corrected pcb layout
Parts:
- removed D5, D6: Q_Thyristor_AGK, Opto-Devices:IRReceiver_Vishay_MINICAST-3pin, symbol Q_Thyristor_AGK
- added D7, D8: Q_Thyristor_KAG, Opto-Devices:IRReceiver_Vishay_MINICAST-3pin, symbol Q_Thyristor_KAG
Connections:
- net GND: now also D7.1 (K), D8.1 (K)
- net at D1.1 (K): now also D7.3 (G)
- net at D4.1 (K): now also D8.3 (G)
- net at C1.1, R2.2: now also D8.2 (A)
- net at C1.2, R1.2: now also D7.2 (A)
Changed lines of the file:
@@
 LIBS:contrib
 LIBS:valves
+LIBS:Class_C_Commuttation_Schematic-cache
 EELAYER 25 0
 EELAYER END
@@
 	8550 5600 8550 5200
 Connection ~ 8500 5600
-$Comp
-L Q_Thyristor_AGK D5
-U 1 1 59E19299
-P 5000 3700
-F 0 "D5" H 5075 3725 50  0000 L CNN
-F 1 "Q_Thyristor_AGK" H 5075 3650 50  0000 L CNN
-F 2 "Opto-Devices:IRReceiver_Vishay_MINICAST-3pin" V 5000 3700 50  0001 C CNN
-F 3 "" V 5000 3700 50  0001 C CNN
-	1    5000 3700
-	1    0    0    -1
-$EndComp
-$Comp
-L Q_Thyristor_AGK D6
-U 1 1 59E19844
-P 6750 3650
-F 0 "D6" H 6825 3675 50  0000 L CNN
-F 1 "Q_Thyristor_AGK" H 6825 3600 50  0000 L CNN
-F 2 "Opto-Devices:IRReceiver_Vishay_MINICAST-3pin" V 6750 3650 50  0001 C CNN
-F 3 "" V 6750 3650 50  0001 C CNN
-	1    6750 3650
-	-1   0    0    -1
-$EndComp
 Wire Wire Line
 	5000 3550 5000 3350
@@
 	8000 5800 8000 5600
 Connection ~ 8000 5600
+$Comp
+L Q_Thyristor_KAG D7
+U 1 1 59E1BB8A
+P 5000 3700
+F 0 "D7" H 5075 3725 50  0000 L CNN
+F 1 "Q_Thyristor_KAG" H 5075 3650 50  0000 L CNN
+F 2 "Opto-Devices:IRReceiver_Vishay_MINICAST-3pin" V 5000 3700 50  0001 C CNN
+F 3 "" V 5000 3700 50  0001 C CNN
+	1    5000 3700
+	1    0    0    -1
+$EndComp
+$Comp
+L Q_Thyristor_KAG D8
+U 1 1 59E1BEC7
+P 6750 3650
+F 0 "D8" H 6825 3675 50  0000 L CNN
+F 1 "Q_Thyristor_KAG" H 6825 3600 50  0000 L CNN
+F 2 "Opto-Devices:IRReceiver_Vishay_MINICAST-3pin" V 6750 3650 50  0001 C CNN
+F 3 "" V 6750 3650 50  0001 C CNN
+	1    6750 3650
+	-1   0    0    -1
+$EndComp
 $EndSCHEMATC
