File: MotionDet/mp2.kicad_pcb (KiCad board)
At the start: 2 copper layers, 152.4 x 101.6 mm, 21 parts, among them J1 +Vcc, J2 -Vcc, J3 Ground, Q1 Q_NMOS_DSG, U1 LM741, U2 LM741, U3 LM741

Commit message: PCB Layout Finalized
Parts:
- moved J3 34.7 mm to (158.8, 137.2)
- moved J2 7.62 mm to (134.6, 121.9)
Routing:
- net GND: track 271.8 -> 211.7 mm
- net Net-(R11-Pad1): track 142.4 -> 150.3 mm
- net /Ve: track 151.3 -> 143.7 mm
Other:
- board text added: "+15v"
- board text added: "-15v"
- board text added: "1"
- board text added: "100k"
- board text added: "10k"
- board text added: "120k"
- board text added: "2.7k"
- board text added: "4.7 k Pot"
- board text added: "4.7k"
- board text added: "5.1k"
- board text added: "5.6k"
- board text added: "PIR Based Motion Detector TE Electronics B1 Sap ID - 11,12,13"
- board text added: "d"
- board text added: "gnd"
- board text added: "n"
- board text added: "p"
- board text added: "s"
